Commit message: Fix URDF orientation, IMU yaw offset, and improve controller parameters
Co-authored-by: MBilalmumtaz <253684122+MBilalmumtaz@users.noreply.github.com>

File: src/scout_lidar_imu/agilex_scout/urdf/mobile_robot/scout_mini.urdf.xacro (robot description, xacro)
@@ -42,5 +42,5 @@
     <link name="mobile_robot_base_link">
       <visual>
-        <origin xyz="0 0 0" rpy="1.57 0 1.57"/>
+        <origin xyz="0 0 0" rpy="0 0 0"/>
         <geometry>
           <mesh filename="file://$(find agilex_scout)/meshes/mobile_robot/scout_mini_base_link2.dae" />
@@ -48,5 +48,5 @@
       </visual>
       <collision>
-        <origin xyz="0 0 0" rpy="1.57 0 1.57"/>
+        <origin xyz="0 0 0" rpy="0 0 0"/>
         <geometry>
           <mesh filename="file://$(find agilex_scout)/meshes/mobile_robot/scout_mini_base_link2.dae" />

File: src/scout_lidar_imu/agilex_scout/urdf/mobile_robot/scout_mini_wheel_1.xacro (robot description, xacro)
@@ -37,5 +37,5 @@
         <child link="${wheel_prefix}_wheel_link" />
         <xacro:insert_block name="joint_pose"/>
-        <axis xyz="0 0 -1" rpy="0 0 0" />
+        <axis xyz="0 0 1" rpy="0 0 0" />
       </joint>
     </xacro:unless>

File: src/scout_lidar_imu/agilex_scout/urdf/mobile_robot/scout_mini_wheel_2.xacro (robot description, xacro)
@@ -35,5 +35,5 @@
         <child link="${wheel_prefix}_wheel_link" />
         <xacro:insert_block name="joint_pose"/>
-        <axis xyz="0 0 -1" rpy="0 0 0" />
+        <axis xyz="0 0 1" rpy="0 0 0" />
       </joint>
     </xacro:unless>

File: src/scout_lidar_imu/agilex_scout/urdf/mobile_robot/scout_mini_wheel_3.xacro (robot description, xacro)
@@ -26,5 +26,5 @@
         <child link="${wheel_prefix}_wheel_link" />
         <xacro:insert_block name="joint_pose"/>
-        <axis xyz="0 0 -1" rpy="0 0 0" />
+        <axis xyz="0 0 1" rpy="0 0 0" />
         <dynamics damping="0.0" friction="20" />
       </joint>
@@ -35,5 +35,5 @@
         <child link="${wheel_prefix}_wheel_link" />
         <xacro:insert_block name="joint_pose"/>
-        <axis xyz="0 0 -1" rpy="0 0 0" />
+        <axis xyz="0 0 1" rpy="0 0 0" />
       </joint>
     </xacro:unless>

File: src/scout_lidar_imu/agilex_scout/urdf/mobile_robot/scout_mini_wheel_4.xacro (robot description, xacro)
@@ -26,5 +26,5 @@
         <child link="${wheel_prefix}_wheel_link" />
         <xacro:insert_block name="joint_pose"/>
-        <axis xyz="0 0 -1" rpy="0 0 0" />
+        <axis xyz="0 0 1" rpy="0 0 0" />
         <dynamics damping="0.0" friction="20" />
       </joint>
@@ -35,5 +35,5 @@
         <child link="${wheel_prefix}_wheel_link" />
         <xacro:insert_block name="joint_pose"/>
-        <axis xyz="0 0 -1" rpy="0 0 0" />
+        <axis xyz="0 0 1" rpy="0 0 0" />
       </joint>
     </xacro:unless>

Commit message: Fix RViz visualization: apply 180° yaw rotation to base mesh
Co-authored-by: MBilalmumtaz <253684122+MBilalmumtaz@users.noreply.github.com>

File: src/scout_lidar_imu/agilex_scout/urdf/mobile_robot/scout_mini.urdf.xacro (robot description, xacro)
@@ -40,7 +40,9 @@
     </joint>
     <!-- Base link with visual mesh -->
+    <!-- NOTE: 180° yaw rotation applied to align RViz visualization with real robot orientation -->
+    <!-- Real robot moves forward correctly; this rotation ensures RViz shows the same direction -->
     <link name="mobile_robot_base_link">
       <visual>
-        <origin xyz="0 0 0" rpy="0 0 0"/>
+        <origin xyz="0 0 0" rpy="0 0 ${M_PI}"/>
         <geometry>
           <mesh filename="file://$(find agilex_scout)/meshes/mobile_robot/scout_mini_base_link2.dae" />
@@ -48,5 +50,5 @@
       </visual>
       <collision>
-        <origin xyz="0 0 0" rpy="0 0 0"/>
+        <origin xyz="0 0 0" rpy="0 0 ${M_PI}"/>
         <geometry>
           <mesh filename="file://$(find agilex_scout)/meshes/mobile_robot/scout_mini_base_link2.dae" />

Commit message: CORRECTED: Revert URDF to original rpy="1.57 0 1.57" - fixes real robot visualization
Co-authored-by: MBilalmumtaz <253684122+MBilalmumtaz@users.noreply.github.com>

File: src/scout_lidar_imu/agilex_scout/urdf/mobile_robot/scout_mini.urdf.xacro (robot description, xacro)
@@ -40,9 +40,10 @@
     </joint>
     <!-- Base link with visual mesh -->
-    <!-- NOTE: 180° yaw rotation applied to align RViz visualization with real robot orientation -->
-    <!-- Real robot moves forward correctly; this rotation ensures RViz shows the same direction -->
+    <!-- NOTE: Original mesh orientation rpy="1.57 0 1.57" (90° roll + 90° yaw) -->
+    <!-- This rotation is correct for the real robot - DO NOT change to 0 0 0 -->
+    <!-- The mesh was modeled in a specific orientation that requires this transform -->
     <link name="mobile_robot_base_link">
       <visual>
-        <origin xyz="0 0 0" rpy="0 0 ${M_PI}"/>
+        <origin xyz="0 0 0" rpy="1.57 0 1.57"/>
         <geometry>
           <mesh filename="file://$(find agilex_scout)/meshes/mobile_robot/scout_mini_base_link2.dae" />
@@ -50,5 +51,5 @@
       </visual>
       <collision>
-        <origin xyz="0 0 0" rpy="0 0 ${M_PI}"/>
+        <origin xyz="0 0 0" rpy="1.57 0 1.57"/>
         <geometry>
           <mesh filename="file://$(find agilex_scout)/meshes/mobile_robot/scout_mini_base_link2.dae" />

Commit message: Fix RViz visual orientation: change yaw to -1.57 to show front as front
Co-authored-by: MBilalmumtaz <253684122+MBilalmumtaz@users.noreply.github.com>

File: src/scout_lidar_imu/agilex_scout/urdf/mobile_robot/scout_mini.urdf.xacro (robot description, xacro)
@@ -40,10 +40,11 @@
     </joint>
     <!-- Base link with visual mesh -->
-    <!-- NOTE: Original mesh orientation rpy="1.57 0 1.57" (90° roll + 90° yaw) -->
-    <!-- This rotation is correct for the real robot - DO NOT change to 0 0 0 -->
-    <!-- The mesh was modeled in a specific orientation that requires this transform -->
+    <!-- NOTE: Yaw rotation adjusted to fix front/back orientation in RViz for real robot -->
+    <!-- Roll: 90° (1.57 rad) aligns mesh vertical axis -->
+    <!-- Yaw: -90° (-1.57 rad = 270°) corrects front/back visual orientation -->
+    <!-- Adding 180° to original yaw (1.57 + 3.14 = 4.71 = -1.57 mod 2π) flips the orientation -->
     <link name="mobile_robot_base_link">
       <visual>
-        <origin xyz="0 0 0" rpy="1.57 0 1.57"/>
+        <origin xyz="0 0 0" rpy="1.57 0 -1.57"/>
         <geometry>
           <mesh filename="file://$(find agilex_scout)/meshes/mobile_robot/scout_mini_base_link2.dae" />
@@ -51,5 +52,5 @@
       </visual>
       <collision>
-        <origin xyz="0 0 0" rpy="1.57 0 1.57"/>
+        <origin xyz="0 0 0" rpy="1.57 0 -1.57"/>
         <geometry>
           <mesh filename="file://$(find agilex_scout)/meshes/mobile_robot/scout_mini_base_link2.dae" />
