Commit message: Fix angular sign correction and TF conflicts for Scout Mini
Co-authored-by: MBilalmumtaz <253684122+MBilalmumtaz@users.noreply.github.com>

File: src/scout_lidar_imu/agilex_scout/urdf/sensors/os1.urdf (robot description, URDF)
Before this commit: robot os1_description, 2 links, 1 joints
Joints:
- removed joint os_sensor_to_imu
- added joint base_to_imu: type fixed, parent mobile_robot_base_link, child imu_link, origin xyz=0 0 0.2 rpy=0 0 -0.94
